Commit message: Bumper spans the full body cylinder height (fixes shelf-ledge wedging)
The bumper was 50mm tall centered at z=0.033 -> it covered only base_link
[0.008, 0.058], missing the bottom ~8mm and top ~8.5mm of the 66.5mm body
cylinder ([0, 0.0665]). A low ledge in that gap -- e.g. a bookcase bottom
shelf -- stops the body but floats under/over the bumper, so no contact
fires and the robot wedges without detecting it.

Make the bumper span the full body height, centered like the body, as a
real consumer-vacuum bumper does: derive bumper_height and bumper_z from
lower_cylinder_height so the front bumper arc always equals the body's
front cylindrical wall and the two can't drift apart. Collision facet
names/indices are unchanged, so the contact-sensor wiring still holds.

Verified: xacro compiles; each bumper facet box is now 0.0665m tall.

Co-Authored-By: Claude Opus 4.8 <noreply@anthropic.com>

File: urdf/params.xacro (robot description, xacro)
@@ -43,6 +43,10 @@
   <xacro:property name="bumper_facets_per_side" value="6"/>
   <xacro:property name="bumper_thickness" value="0.010"/> <!-- radial; outer face ~5mm proud -->
-  <xacro:property name="bumper_height" value="0.050"/>
-  <xacro:property name="bumper_z" value="0.033"/>     <!-- center height in base_link frame -->
+  <!-- Bumper spans the FULL body cylinder height, centered on it (like a consumer
+       vacuum), so a low ledge the body can hit (e.g. a bookcase bottom shelf)
+       always contacts the bumper instead of wedging in the gap above or below it.
+       Derived from lower_cylinder_height so the two can never drift apart. -->
+  <xacro:property name="bumper_height" value="${lower_cylinder_height}"/>
+  <xacro:property name="bumper_z" value="${lower_cylinder_height/2}"/>  <!-- = body cylinder center, base_link frame -->
   <xacro:property name="DEG2RAD" value="0.0174533"/>
 </robot>

Commit message: Add left/right side distance sensors (short-range wall sensors)
Model a short-range IR/ToF side wall sensor on each side of the body, aimed
straight out (perpendicular to forward) at the body's mid-height. Perpendicular
aim reads wall distance directly abeam -- the basis for distance-keeping wall
following, the natural step past the current bump-and-turn. gz-sim has no native
Range/sonar sensor, so each is a gpu_lidar publishing sensor_msgs/LaserScan; on
the physical robot these map to ToF -> sensor_msgs/Range (a sim/real difference
like the bumpers).

- params.xacro: side-sensor geometry + beam, all tunable (min/max range 0.02/0.5 m,
  aim, mount x/z, update rate, samples, FOV).
- robot.urdf.xacro: side_range_sensor macro -> range_left_link / range_right_link
  on the body side edges (fixed joints, tiny visual + inertia, no collision so the
  bumper collision lumping is unchanged -- test_bumper_wiring still passes).
- plugins.xacro: a gpu_lidar per side. Two gz-specific points learned the hard way
  and documented inline:
    * the sensor pose is baked relative to base_link (the canonical link) rather
      than the fixed-joint-lumped sensor-link frame, so the ray aim is robust to
      URDF->SDF lumping;
    * samples must be >= 2 -- gz computes angle_step = (max-min)/(samples-1), so
      samples=1 yields angle_step=NaN and the ray never fires. Modelled as a narrow
      3-sample, 1-degree cone (a real ToF's small FOV); a consumer takes min(ranges)
      as the distance.
- gz_bridge.yaml: bridge range_left / range_right (gz.msgs.LaserScan -> LaserScan).

Verified: xacro compiles, URDF->SDF converts, sensor world_pose is correct
(y +/-0.1745, z 0.046, yaw +/-90 deg), angle_step is finite, and the bridge config
is valid. Live range VALUES could not be read in the headless CI container --
gpu_lidar needs a GPU/EGL render context, so /scan reads all-inf there too -- so
confirm /range_left and /range_right in a rendered sim.

Co-Authored-By: Claude Opus 4.8 <noreply@anthropic.com>

File: urdf/params.xacro (robot description, xacro)
@@ -49,4 +49,26 @@
   <xacro:property name="bumper_height" value="${lower_cylinder_height}"/>
   <xacro:property name="bumper_z" value="${lower_cylinder_height/2}"/>  <!-- = body cylinder center, base_link frame -->
+  <!-- ****************** SIDE DISTANCE SENSORS ****************** -->
+  <!-- Left/right short-range wall sensors. Modelled as a single-ray gpu_lidar
+       (gz-sim has no native Range/ToF sensor) aimed straight out to the side,
+       perpendicular to forward, at the body's mid-height on each side edge. That
+       aim reads the wall distance directly abeam, the basis for distance-keeping
+       wall following. On the physical robot this maps to a ToF (sensor_msgs/Range);
+       in sim it is a 1-beam sensor_msgs/LaserScan. All values below are tunable. -->
+  <xacro:property name="range_sensor_min" value="0.02"/>          <!-- m: closest reading -->
+  <xacro:property name="range_sensor_max" value="0.50"/>          <!-- m: beyond this reads as no wall -->
+  <xacro:property name="range_sensor_resolution" value="0.005"/>  <!-- m -->
+  <xacro:property name="range_sensor_angle_deg" value="90.0"/>    <!-- deg from forward; 90 = straight out to the side -->
+  <xacro:property name="range_sensor_x" value="0.0"/>             <!-- fore/aft mount offset along the side -->
+  <xacro:property name="range_sensor_z" value="${lower_cylinder_height/2}"/> <!-- body mid-height, base_link frame -->
+  <xacro:property name="range_sensor_update_rate" value="20"/>    <!-- Hz -->
+  <xacro:property name="range_sensor_size" value="0.012"/>        <!-- visual cube edge (m) -->
+  <xacro:property name="range_sensor_mass" value="0.005"/>        <!-- kg, negligible -->
+  <!-- gz-sim's gpu_lidar needs 2 or more samples: angle_step = (max-min)/(samples-1),
+       so samples=1 divides by zero (angle_step = NaN, the ray never fires). Model
+       the beam as a narrow few-sample cone instead, like a real ToF's small field
+       of view; a consumer takes the nearest (min) range as THE distance. -->
+  <xacro:property name="range_sensor_samples" value="3"/>         <!-- rays across the FOV (2 or more) -->
+  <xacro:property name="range_sensor_fov_deg" value="1.0"/>       <!-- total beam FOV (deg) -->
   <xacro:property name="DEG2RAD" value="0.0174533"/>
 </robot>

File: urdf/plugins.xacro (robot description, xacro)
@@ -108,3 +108,45 @@
     </sensor>
   </gazebo>
+  <!-- Left/right side distance sensors: a single ray straight out to the side,
+       modelling a short-range IR/ToF wall sensor. gz-sim publishes gz.msgs.LaserScan
+       (one beam) on <topic>, which config/gz_bridge.yaml bridges to sensor_msgs/
+       LaserScan. Attached to the sensor link (see robot.urdf.xacro); like the
+       gpu_lidar above, gz honours <topic> (unlike the contact sensors). -->
+  <xacro:macro name="side_range_plugin" params="prefix side_sign">
+    <gazebo reference="base_link">
+      <sensor name="${prefix}" type="gpu_lidar">
+        <!-- Pose baked relative to base_link (the canonical link, unaffected by
+             fixed-joint lumping) so the ray aim does not depend on the lumped
+             sensor-link frame orientation. Matches the ${prefix}_link URDF joint. -->
+        <pose relative_to="base_link">${range_sensor_x} ${side_sign * base_diameter/2} ${range_sensor_z} 0 0 ${side_sign * range_sensor_angle_deg * DEG2RAD}</pose>
+        <update_rate>${range_sensor_update_rate}</update_rate>
+        <topic>${prefix}</topic>
+        <gz_frame_id>${prefix}_link</gz_frame_id>
+        <ray>
+          <scan>
+            <horizontal>
+              <samples>${range_sensor_samples}</samples>
+              <resolution>1</resolution>
+              <min_angle>${-range_sensor_fov_deg/2 * DEG2RAD}</min_angle>
+              <max_angle>${ range_sensor_fov_deg/2 * DEG2RAD}</max_angle>
+            </horizontal>
+          </scan>
+          <range>
+            <min>${range_sensor_min}</min>
+            <max>${range_sensor_max}</max>
+            <resolution>${range_sensor_resolution}</resolution>
+          </range>
+          <noise>
+            <type>gaussian</type>
+            <mean>0.0</mean>
+            <stddev>0.005</stddev>
+          </noise>
+        </ray>
+        <always_on>1</always_on>
+        <visualize>true</visualize>
+      </sensor>
+    </gazebo>
+  </xacro:macro>
+  <xacro:side_range_plugin prefix="range_left" side_sign="1"/>
+  <xacro:side_range_plugin prefix="range_right" side_sign="-1"/>
 </robot>

File: urdf/robot.urdf.xacro (robot description, xacro)
@@ -34,4 +34,27 @@
       <xacro:bumper_arc prefix="${prefix}" a0="${a0}" n="${n}" i="${i + 1}"/>
     </xacro:if>
+  </xacro:macro>
+  <!-- One side distance sensor: a small link on the body side edge whose +X axis
+       (the single ray's direction) is aimed outward. side_sign = +1 left (+Y),
+       -1 right (-Y); range_sensor_angle_deg is measured from forward (90 = straight
+       out). The matching gpu_lidar sensor is in plugins.xacro. -->
+  <xacro:macro name="side_range_sensor" params="prefix side_sign">
+    <joint name="${prefix}_joint" type="fixed">
+      <parent link="base_link"/>
+      <child link="${prefix}_link"/>
+      <origin xyz="${range_sensor_x} ${side_sign * base_diameter/2} ${range_sensor_z}"
+              rpy="0 0 ${side_sign * range_sensor_angle_deg * DEG2RAD}"/>
+    </joint>
+    <link name="${prefix}_link">
+      <visual>
+        <origin xyz="0 0 0" rpy="0 0 0"/>
+        <geometry>
+          <box size="${range_sensor_size} ${range_sensor_size} ${range_sensor_size}"/>
+        </geometry>
+        <material name="dark"/>
+      </visual>
+      <xacro:solid_box_inertia m="${range_sensor_mass}"
+        x="${range_sensor_size}" y="${range_sensor_size}" z="${range_sensor_size}"/>
+    </link>
   </xacro:macro>
   <link name="base_footprint"/>
@@ -157,3 +180,6 @@
     <xacro:solid_cylinder_inertia m="${laser_puck_mass}" r="${laser_puck_diameter/2}" h="${laser_puck_height}"/>
   </link>
+  <!-- Left/right side distance sensors (short-range wall sensors) -->
+  <xacro:side_range_sensor prefix="range_left" side_sign="1"/>
+  <xacro:side_range_sensor prefix="range_right" side_sign="-1"/>
 </robot>

Commit message: Add front multizone ToF depth sensor and front stereo cameras
Front sensor suite on the body front face, at mid-height, front & center:

- tof_front: a front-facing depth grid modelling two VL53L7CX multizone ToF
  arrays (each 8x8 zones, 60 deg H) aimed +/-30 deg, so together 120 deg. One
  gpu_lidar with a 16 (=8+8) x 8 ray grid over 120 deg H x 60 deg V; each ray is
  a zone distance. Published as /tof_front/points (PointCloud2, 128 pts).

- camera_left / camera_right: two RGB cameras (OV5647-equivalent, VGA 640x480,
  120 deg HFoV) flanking the ToF on a compact 50 mm stereo base, for obstacle
  recognition and future stereo depth. Each has a REP-103 optical frame the image
  is stamped in. Published as /camera_{left,right}/image + /camera_info. URDF +
  topics only for now; no stereo processing yet.

All geometry/optics are tunable params in params.xacro; sensor blocks in
plugins.xacro; ROS bridging in config/gz_bridge.yaml. The new links are
visual-only (no collisions), so bumper collision indices are unchanged.

Verified in the jazzy container: xacro -> gz sdf converts clean, all 8 sensors
present (tof_front 16x8, cameras 640x480 @ 120 deg), gz topic names match the
bridge (/tof_front/points, /camera_*/image, /camera_*/camera_info), and
test/test_bumper_wiring.py still passes. Live depth/image data needs the GPU
render path (works on the sim host; not reproducible in this headless container).

Co-Authored-By: Claude Opus 4.8 <noreply@anthropic.com>

File: urdf/params.xacro (robot description, xacro)
@@ -71,4 +71,40 @@
   <xacro:property name="range_sensor_samples" value="3"/>         <!-- rays across the FOV (2 or more) -->
   <xacro:property name="range_sensor_fov_deg" value="1.0"/>       <!-- total beam FOV (deg) -->
+  <!-- ****************** FRONT DISTANCE SENSOR (multizone ToF) ****************** -->
+  <!-- Front-facing depth grid, front & center. Models TWO VL53L7CX multizone ToF
+       sensors (each 8x8 zones, 60 deg horizontal FoV) mounted one aimed 30 deg left
+       and one 30 deg right, so together they span 120 deg. Represented as ONE
+       gpu_lidar with a 16 (= 8 + 8) x 8 ray grid over 120 deg H x 60 deg V, where
+       each ray is a zone distance. Published as a PointCloud2 (128 points); on the
+       physical robot these are per-zone ToF ranges. All values tunable. -->
+  <xacro:property name="tof_front_h_samples" value="16"/>          <!-- 8 + 8 zones across -->
+  <xacro:property name="tof_front_v_samples" value="8"/>           <!-- 8 zones tall -->
+  <xacro:property name="tof_front_hfov_deg" value="120.0"/>        <!-- 2 x 60 deg -->
+  <xacro:property name="tof_front_vfov_deg" value="60.0"/>         <!-- one sensor's vertical FoV -->
+  <xacro:property name="tof_front_min" value="0.02"/>              <!-- m -->
+  <xacro:property name="tof_front_max" value="4.0"/>               <!-- m: VL53L7CX long range -->
+  <xacro:property name="tof_front_resolution" value="0.005"/>      <!-- m -->
+  <xacro:property name="tof_front_update_rate" value="15"/>        <!-- Hz -->
+  <xacro:property name="tof_front_x" value="${base_diameter/2}"/>  <!-- front surface -->
+  <xacro:property name="tof_front_z" value="${lower_cylinder_height/2}"/> <!-- mid-height -->
+  <xacro:property name="tof_front_size" value="0.012"/>            <!-- visual cube edge (m) -->
+  <xacro:property name="tof_front_mass" value="0.005"/>            <!-- kg, negligible -->
+  <!-- ****************** FRONT STEREO CAMERAS (OV5647) ****************** -->
+  <!-- Two RGB cameras, front & center, flanking the ToF sensor left/right, for
+       obstacle recognition and future stereo depth. VGA, wide FoV. The stereo base
+       is small on purpose (we only need coarse obstacle depth). URDF + camera topics
+       only for now, no stereo processing yet. Each has a REP-103 optical frame
+       (z-forward, x-right, y-down) that the image is published in. Tunable. -->
+  <xacro:property name="camera_width" value="640"/>                <!-- VGA -->
+  <xacro:property name="camera_height" value="480"/>
+  <xacro:property name="camera_hfov_deg" value="120.0"/>
+  <xacro:property name="camera_near" value="0.02"/>                <!-- m -->
+  <xacro:property name="camera_far" value="10.0"/>                 <!-- m -->
+  <xacro:property name="camera_update_rate" value="15"/>           <!-- Hz -->
+  <xacro:property name="camera_baseline" value="0.05"/>            <!-- m: compact stereo base -->
+  <xacro:property name="camera_x" value="${base_diameter/2}"/>     <!-- front surface -->
+  <xacro:property name="camera_z" value="${lower_cylinder_height/2}"/> <!-- mid-height, flanking the ToF -->
+  <xacro:property name="camera_size" value="0.010"/>               <!-- visual cube edge (m) -->
+  <xacro:property name="camera_mass" value="0.005"/>               <!-- kg, negligible -->
   <xacro:property name="DEG2RAD" value="0.0174533"/>
 </robot>

File: urdf/plugins.xacro (robot description, xacro)
@@ -150,3 +150,74 @@
   <xacro:side_range_plugin prefix="range_left" side_sign="1"/>
   <xacro:side_range_plugin prefix="range_right" side_sign="-1"/>
+  <!-- Front multizone ToF depth sensor: a 16 (= 8 + 8) x 8 gpu_lidar ray grid over
+       120 deg H x 60 deg V, front & center, modelling two VL53L7CX (each 8x8, 60
+       deg) aimed +/-30 deg. gz publishes a gz.msgs.PointCloudPacked on tof_front/
+       points, which config/gz_bridge.yaml bridges to sensor_msgs/PointCloud2. -->
+  <gazebo reference="tof_front_link">
+    <sensor name="tof_front" type="gpu_lidar">
+      <pose relative_to="tof_front_link">0 0 0 0 0 0</pose>
+      <update_rate>${tof_front_update_rate}</update_rate>
+      <topic>tof_front</topic>
+      <gz_frame_id>tof_front_link</gz_frame_id>
+      <ray>
+        <scan>
+          <horizontal>
+            <samples>${tof_front_h_samples}</samples>
+            <resolution>1</resolution>
+            <min_angle>${-tof_front_hfov_deg/2 * DEG2RAD}</min_angle>
+            <max_angle>${ tof_front_hfov_deg/2 * DEG2RAD}</max_angle>
+          </horizontal>
+          <vertical>
+            <samples>${tof_front_v_samples}</samples>
+            <resolution>1</resolution>
+            <min_angle>${-tof_front_vfov_deg/2 * DEG2RAD}</min_angle>
+            <max_angle>${ tof_front_vfov_deg/2 * DEG2RAD}</max_angle>
+          </vertical>
+        </scan>
+        <range>
+          <min>${tof_front_min}</min>
+          <max>${tof_front_max}</max>
+          <resolution>${tof_front_resolution}</resolution>
+        </range>
+        <noise>
+          <type>gaussian</type>
+          <mean>0.0</mean>
+          <stddev>0.005</stddev>
+        </noise>
+      </ray>
+      <always_on>1</always_on>
+      <visualize>true</visualize>
+    </sensor>
+  </gazebo>
+  <!-- One front RGB camera (OV5647-equivalent), VGA, wide FoV. gz publishes
+       gz.msgs.Image on <topic> and gz.msgs.CameraInfo on the sibling camera_info
+       topic (the /image suffix -> /camera_info); config/gz_bridge.yaml bridges both.
+       The image is stamped in the ROS optical frame. -->
+  <xacro:macro name="camera_plugin" params="side">
+    <gazebo reference="camera_${side}_link">
+      <sensor name="camera_${side}" type="camera">
+        <pose relative_to="camera_${side}_link">0 0 0 0 0 0</pose>
+        <update_rate>${camera_update_rate}</update_rate>
+        <topic>camera_${side}/image</topic>
+        <gz_frame_id>camera_${side}_optical_frame</gz_frame_id>
+        <camera>
+          <horizontal_fov>${camera_hfov_deg * DEG2RAD}</horizontal_fov>
+          <image>
+            <width>${camera_width}</width>
+            <height>${camera_height}</height>
+            <format>R8G8B8</format>
+          </image>
+          <clip>
+            <near>${camera_near}</near>
+            <far>${camera_far}</far>
+          </clip>
+          <optical_frame_id>camera_${side}_optical_frame</optical_frame_id>
+        </camera>
+        <always_on>1</always_on>
+        <visualize>true</visualize>
+      </sensor>
+    </gazebo>
+  </xacro:macro>
+  <xacro:camera_plugin side="left"/>
+  <xacro:camera_plugin side="right"/>
 </robot>

File: urdf/robot.urdf.xacro (robot description, xacro)
@@ -58,4 +58,53 @@
     </link>
   </xacro:macro>
+  <!-- Front multizone ToF: a small forward-facing link at body mid-height, front
+       center. Its +X is the depth-grid boresight; the 16x8 ray sensor is in
+       plugins.xacro. Visual is a wide box hinting at the two ToF modules. -->
+  <xacro:macro name="front_tof_sensor">
+    <joint name="tof_front_joint" type="fixed">
+      <parent link="base_link"/>
+      <child link="tof_front_link"/>
+      <origin xyz="${tof_front_x} 0 ${tof_front_z}" rpy="0 0 0"/>
+    </joint>
+    <link name="tof_front_link">
+      <visual>
+        <origin xyz="0 0 0" rpy="0 0 0"/>
+        <geometry>
+          <box size="${tof_front_size} ${2*tof_front_size} ${tof_front_size}"/>
+        </geometry>
+        <material name="dark"/>
+      </visual>
+      <xacro:solid_box_inertia m="${tof_front_mass}"
+        x="${tof_front_size}" y="${2*tof_front_size}" z="${tof_front_size}"/>
+    </link>
+  </xacro:macro>
+  <!-- One front RGB camera flanking the ToF, plus a ROS optical frame (REP-103:
+       x right, y down, z forward) the image is published in. side_sign = +1 left
+       (+Y), -1 right (-Y). The gz camera sensor is in plugins.xacro. -->
+  <xacro:macro name="stereo_camera" params="side side_sign">
+    <joint name="camera_${side}_joint" type="fixed">
+      <parent link="base_link"/>
+      <child link="camera_${side}_link"/>
+      <origin xyz="${camera_x} ${side_sign * camera_baseline/2} ${camera_z}"
+              rpy="0 0 0"/>
+    </joint>
+    <link name="camera_${side}_link">
+      <visual>
+        <origin xyz="0 0 0" rpy="0 0 0"/>
+        <geometry>
+          <box size="${camera_size} ${camera_size} ${camera_size}"/>
+        </geometry>
+        <material name="dark"/>
+      </visual>
+      <xacro:solid_box_inertia m="${camera_mass}"
+        x="${camera_size}" y="${camera_size}" z="${camera_size}"/>
+    </link>
+    <joint name="camera_${side}_optical_joint" type="fixed">
+      <parent link="camera_${side}_link"/>
+      <child link="camera_${side}_optical_frame"/>
+      <origin xyz="0 0 0" rpy="${-pi/2} 0 ${-pi/2}"/>
+    </joint>
+    <link name="camera_${side}_optical_frame"/>
+  </xacro:macro>
   <link name="base_footprint"/>
   <joint name="base_joint" type="fixed">
@@ -183,3 +232,8 @@
   <xacro:side_range_sensor prefix="range_left" side_sign="1"/>
   <xacro:side_range_sensor prefix="range_right" side_sign="-1"/>
+  <!-- Front multizone ToF depth sensor (front & center) -->
+  <xacro:front_tof_sensor/>
+  <!-- Front stereo cameras, flanking the ToF left/right -->
+  <xacro:stereo_camera side="left" side_sign="1"/>
+  <xacro:stereo_camera side="right" side_sign="-1"/>
 </robot>
