Commit message: Add a simulated IMU (gyro + accelerometer) -> /imu
The sim had no IMU (only the physical robot published /imu, and ekf.yaml already
expects it). Adds a gz imu sensor at a new imu_link near the body center,
bridged to sensor_msgs/Imu on /imu.

Orientation is DISABLED so /imu carries angular velocity + linear acceleration
only, like the gyro+accel hardware IMU the EKF is tuned for (it fuses the yaw
rate). The sim leaves the orientation field unset (zero quaternion); the hardware
bridge instead flags no-orientation with orientation_covariance[0] = -1.

Like the contact sensors, the gz imu sensor needs the world-level
gz-sim-imu-system. oomwoo_gazebo living_room.world already loads it; test_room.world
gets it in a companion commit. All values are tunable params in params.xacro.
README sensor table + params list updated.

Verified in the jazzy container: /imu publishes at rest with accel.z ~= 9.78
(gravity), gyro ~= 0, and the configured noise covariances; the bumper wiring
test still passes (imu_link is visual-only, no collisions).

Co-Authored-By: Claude Opus 4.8 <noreply@anthropic.com>

File: urdf/params.xacro (robot description, xacro)
@@ -107,4 +107,17 @@
   <xacro:property name="camera_size" value="0.010"/>               <!-- visual cube edge (m) -->
   <xacro:property name="camera_mass" value="0.005"/>               <!-- kg, negligible -->
+  <!-- ****************** IMU ****************** -->
+  <!-- 6-axis IMU (gyro + accelerometer) near the body center, mirroring the
+       physical robot's board IMU. Orientation is DISABLED (see plugins.xacro) so
+       /imu carries only angular_velocity + linear_acceleration, exactly like the
+       SangamIO/Proscenic gyro the EKF expects (config/ekf.yaml). Tunable. -->
+  <xacro:property name="imu_x" value="0.0"/>
+  <xacro:property name="imu_y" value="0.0"/>
+  <xacro:property name="imu_z" value="${lower_cylinder_height/2}"/> <!-- body mid-height -->
+  <xacro:property name="imu_update_rate" value="100"/>             <!-- Hz -->
+  <xacro:property name="imu_gyro_noise" value="0.0002"/>           <!-- rad/s stddev (MEMS-ish) -->
+  <xacro:property name="imu_accel_noise" value="0.017"/>           <!-- m/s^2 stddev -->
+  <xacro:property name="imu_size" value="0.010"/>                  <!-- visual cube edge (m) -->
+  <xacro:property name="imu_mass" value="0.005"/>                  <!-- kg, negligible -->
   <xacro:property name="DEG2RAD" value="0.0174533"/>
 </robot>

File: urdf/plugins.xacro (robot description, xacro)
@@ -256,3 +256,34 @@
   <xacro:camera_plugin side="left"/>
   <xacro:camera_plugin side="right"/>
+  <!-- IMU: 6-axis (gyro + accelerometer) at imu_link, near the body center. gz
+       publishes gz.msgs.IMU on <topic>, bridged to sensor_msgs/Imu. Orientation
+       is DISABLED so /imu carries angular velocity + linear acceleration only,
+       like the physical robot's IMU (the EKF fuses the yaw rate, config/ekf.yaml).
+       The sim leaves the orientation field unset (a zero quaternion); the hardware
+       bridge instead flags "no orientation" with orientation_covariance[0] = -1.
+       Like the contact sensors, this needs the world to load the world-level
+       gz-sim-imu-system; oomwoo_gazebo living_room.world and oomwoo_sim_support
+       test_room.world both do (an IMU-less world leaves /imu silent). -->
+  <gazebo reference="imu_link">
+    <sensor name="imu" type="imu">
+      <pose relative_to="imu_link">0 0 0 0 0 0</pose>
+      <update_rate>${imu_update_rate}</update_rate>
+      <topic>imu</topic>
+      <gz_frame_id>imu_link</gz_frame_id>
+      <imu>
+        <enable_orientation>false</enable_orientation>
+        <angular_velocity>
+          <x><noise type="gaussian"><mean>0.0</mean><stddev>${imu_gyro_noise}</stddev></noise></x>
+          <y><noise type="gaussian"><mean>0.0</mean><stddev>${imu_gyro_noise}</stddev></noise></y>
+          <z><noise type="gaussian"><mean>0.0</mean><stddev>${imu_gyro_noise}</stddev></noise></z>
+        </angular_velocity>
+        <linear_acceleration>
+          <x><noise type="gaussian"><mean>0.0</mean><stddev>${imu_accel_noise}</stddev></noise></x>
+          <y><noise type="gaussian"><mean>0.0</mean><stddev>${imu_accel_noise}</stddev></noise></y>
+          <z><noise type="gaussian"><mean>0.0</mean><stddev>${imu_accel_noise}</stddev></noise></z>
+        </linear_acceleration>
+      </imu>
+      <always_on>1</always_on>
+    </sensor>
+  </gazebo>
 </robot>

File: urdf/robot.urdf.xacro (robot description, xacro)
@@ -237,3 +237,20 @@
   <xacro:stereo_camera side="left" side_sign="1"/>
   <xacro:stereo_camera side="right" side_sign="-1"/>
+  <!-- IMU (gyro + accelerometer), near the body center -->
+  <joint name="imu_joint" type="fixed">
+    <parent link="base_link"/>
+    <child link="imu_link"/>
+    <origin xyz="${imu_x} ${imu_y} ${imu_z}" rpy="0 0 0"/>
+  </joint>
+  <link name="imu_link">
+    <visual>
+      <origin xyz="0 0 0" rpy="0 0 0"/>
+      <geometry>
+        <box size="${imu_size} ${imu_size} ${imu_size}"/>
+      </geometry>
+      <material name="orange"/>
+    </visual>
+    <xacro:solid_box_inertia m="${imu_mass}"
+      x="${imu_size}" y="${imu_size}" z="${imu_size}"/>
+  </link>
 </robot>
